File: hardware/buckbench-cc20.kicad_sch (KiCad schematic)
At the start: 73 parts, among them J1 VSTUP 24 V DC, J2 VÝSTUP, Q1 BC337, Q2 BC337, Q3 BC337, Q4 BC337, Q5 BC547, SW1 SÍŤOVÝ VYPÍNAČ, SW2 U/I (MODE), SW3 VÝSTUP ON/OFF, U1 LM358

Commit message: Přejmenování projektu na Buckbench-CC20
Co-Authored-By: Claude Opus 5.5 <noreply@anthropic.com>
Claude-Session: https://claude.ai/code/session_01Ssrj2kgLuwDYsWDSUoWqnJ
Other:
- title: BuckBench – mini laboratorní zdroj (LM2596S + STM32) -> Buckbench-CC20 – laboratorní zdroj 20 V / 2 A
